File: Designs/KiCAD Files/WRECtangleVersions/V4.1/Wrectangle-V4/24V-PowerCircuit.kicad_sch (KiCad schematic)
At the start: 26 parts, among them M1-24V1 60V, M2-24V1 40V, U7 TPS43060RTER

Commit message: all but one ERC error????
MAYBE??
Connections:
- net 0 renamed GND
Changed lines of the file:
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@@
-	)
-	(junction
-		(at 53.34 72.39)
-		(diameter 0)
-		(color 0 0 0 0)
 	)
 	(junction
@@
 	(wire
 		(pts
-			(xy 50.8 72.39) (xy 53.34 72.39)
-		)
-		(stroke
-			(width 0)
-			(type default)
-		)
-	)
-	(wire
-		(pts
 			(xy 53.34 139.7) (xy 76.2 139.7)
 		)
@@
 	(wire
 		(pts
-			(xy 53.34 72.39) (xy 53.34 62.23)
+			(xy 53.34 62.23) (xy 53.34 139.7)
 		)
 		(stroke
@@
 		(pts
 			(xy 255.27 45.72) (xy 236.22 45.72)
-		)
-		(stroke
-			(width 0)
-			(type default)
-		)
-	)
-	(wire
-		(pts
-			(xy 53.34 139.7) (xy 53.34 72.39)
 		)
 		(stroke
@@
 					(unit 1)
 				)
-			)
-		)
-	)
-	(symbol
-		(lib_id "Simulation_SPICE:0")
-		(at 50.8 72.39 270)
-		(unit 1)
-		(exclude_from_sim no)
-		(in_bom yes)
-		(on_board yes)
-		(dnp no)
-		(fields_autoplaced yes)
-		(property "Reference" "#GND01"
-			(at 45.72 72.39 0)
-			(effects
-				(font
-					(size 1.27 1.27)
-				)
-				(hide yes)
-			)
-		)
-		(property "Value" "0"
-			(at 52.07 72.3899 90)
-			(effects
-				(font
-					(size 1.27 1.27)
-				)
-				(justify left)
-			)
-		)
-		(property "Footprint" ""
-			(at 50.8 72.39 0)
-			(effects
-				(font
-					(size 1.27 1.27)
-				)
-				(hide yes)
-			)
-		)
-		(property "Datasheet" "https://ngspice.sourceforge.io/docs/ngspice-html-manual/manual.xhtml#subsec_Circuit_elements__device"
-			(at 40.64 72.39 0)
-			(effects
-				(font
-					(size 1.27 1.27)
-				)
-				(hide yes)
-			)
-		)
-		(property "Description" "0V reference potential for simulation"
-			(at 43.18 72.39 0)
-			(effects
-				(font
-					(size 1.27 1.27)
-				)
-				(hide yes)
-			)
-		)
-		(pin "1"
-		)
-		(instances
-			(project ""
-				(path "/999a87cf-6a03-4be4-a445-b5341a1dddf0/a54ed999-f025-4f35-b083-b61c3d192ac9"
-					(reference "#GND01")
-					(unit 1)
-				)

Commit message: Error Free!
yay.
Parts:
- R13-24V1, R14-24V1: value 10 -> 10Ω
- Rfbb-24V1: value 11k -> 11kΩ
- Rfbt-24V1: value 205k -> 205kΩ
- Rpg-24V1: value 100k -> 100kΩ
- Rsns1-24V1, Rsns2-24V1: value 7m -> 7mΩ 1W
Changed lines of the file:
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@@
-	(wire
-		(pts
-			(xy 38.1 163.83) (xy 64.77 163.83)
-		)
-		(stroke
-			(width 0)
-			(type default)
-		)
-	)
 	(wire
 		(pts
@@
 	(wire
 		(pts
-			(xy 38.1 157.48) (xy 38.1 163.83)
-		)
-		(stroke
-			(width 0)
-			(type default)
-		)
-	)
-	(wire
-		(pts
 			(xy 255.27 45.72) (xy 236.22 45.72)
 		)
@@
 		)
 	)
-	(global_label "VBAT"
+	(global_label "24VCC"
 		(shape input)
-		(at 64.77 163.83 0)
+		(at 255.27 45.72 0)
 		(fields_autoplaced yes)
 		(effects
@@
 		)
 		(property "Intersheetrefs" "${INTERSHEET_REFS}"
-			(at 72.17 163.83 0)
+			(at 264.3028 45.72 0)
 			(effects
 				(font
@@
 		)
 	)
-	(global_label "24VCC"
+	(global_label "VBAT"
 		(shape input)
-		(at 255.27 45.72 0)
+		(at 53.34 54.61 180)
 		(fields_autoplaced yes)
 		(effects
@@
 				(size 1.27 1.27)
 			)
-			(justify left)
-		)
-		(property "Intersheetrefs" "${INTERSHEET_REFS}"
-			(at 264.3028 45.72 0)
-			(effects
-				(font
-					(size 1.27 1.27)
-				)
-				(justify left)
-				(hide yes)
-			)
-		)
-	)
-	(global_label "VBAT"
-		(shape input)
-		(at 53.34 54.61 180)
-		(fields_autoplaced yes)
-		(effects
-			(font
-				(size 1.27 1.27)
-			)
 			(justify right)
 		)
@@
 			)
 		)
-		(property "Value" "10"
+		(property "Value" "10Ω"
 			(at 101.6 63.4999 0)
 			(effects
@@
 			)
 		)
-		(property "Value" "7m"
+		(property "Value" "7mΩ 1W"
 			(at 113.03 41.91 90)
 			(effects
@@
 			)
 		)
-		(property "Value" "100k"
+		(property "Value" "100kΩ"
 			(at 196.85 73.6599 0)
 			(effects
@@
 			)
 		)
-		(property "Value" "205k"
+		(property "Value" "205kΩ"
 			(at 238.76 64.7699 0)
 			(effects
@@
 			)
 		)
-		(property "Value" "11k"
+		(property "Value" "11kΩ"
 			(at 238.76 78.7399 0)
 			(effects
@@
 			)
 		)
-		(property "Value" "10"
+		(property "Value" "10Ω"
 			(at 121.92 63.4999 0)
 			(effects
@@
 	)
 	(symbol
-		(lib_id "power:+12V")
-		(at 38.1 157.48 0)
-		(unit 1)
-		(exclude_from_sim no)
-		(in_bom yes)
-		(on_board yes)
-		(dnp no)
-		(fields_autoplaced yes)
-		(property "Reference" "#PWR076"
-			(at 38.1 161.29 0)
-			(effects
-				(font
-					(size 1.27 1.27)
-				)
-				(hide yes)
-			)
-		)
-		(property "Value" "+12V"
-			(at 38.1 152.4 0)
-			(effects
-				(font
-					(size 1.27 1.27)
-				)
-			)
-		)
-		(property "Footprint" ""
-			(at 38.1 157.48 0)
-			(effects
-				(font
-					(size 1.27 1.27)
-				)
-				(hide yes)
-			)
-		)
-		(property "Datasheet" ""
-			(at 38.1 157.48 0)
-			(effects
-				(font
-					(size 1.27 1.27)
-				)
-				(hide yes)
-			)
-		)
-		(property "Description" "Power symbol creates a global label with name \"+12V\""
-			(at 38.1 157.48 0)
-			(effects
-				(font
-					(size 1.27 1.27)
-				)
-				(hide yes)
-			)
-		)
-		(pin "1"
-		)
-		(instances
-			(project ""
-				(path "/999a87cf-6a03-4be4-a445-b5341a1dddf0/a54ed999-f025-4f35-b083-b61c3d192ac9"
-					(reference "#PWR076")
-					(unit 1)
-				)
-			)
-		)
-	)
-	(symbol
 		(lib_id "power:GND")
 		(at 132.08 67.31 0)
@@
 			)
 		)
-		(property "Value" "7m"
+		(property "Value" "7mΩ 1W"
 			(at 111.76 53.34 90)
 			(effects
