File: Designs/KiCAD Files/WRECtangleVersions/V4.1/Wrectangle-V4/power.kicad_sch (KiCad schematic)
At the start: 20 parts, among them J1 Conn_01x02_Socket, U6 TPS55289RYQR

Commit message: all but one ERC error????
MAYBE??
Changed lines of the file:
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@@
-	)
-	(junction
-		(at 63.5 63.5)
-		(diameter 0)
-		(color 0 0 0 0)
 	)
 	(junction
@@
 	)
 	(junction
+		(at 76.2 68.58)
+		(diameter 0)
+		(color 0 0 0 0)
+	)
+	(junction
 		(at 48.26 58.42)
 		(diameter 0)
@@
 	)
 	(junction
+		(at 63.5 68.58)
+		(diameter 0)
+		(color 0 0 0 0)
+	)
+	(junction
 		(at 88.9 50.8)
 		(diameter 0)
@@
 	)
 	(junction
+		(at 88.9 68.58)
+		(diameter 0)
+		(color 0 0 0 0)
+	)
+	(junction
 		(at 234.95 120.65)
 		(diameter 0)
@@
 	)
 	(junction
-		(at 88.9 63.5)
-		(diameter 0)
-		(color 0 0 0 0)
-	)
-	(junction
 		(at 207.01 110.49)
 		(diameter 0)
@@
 	(junction
 		(at 107.95 139.7)
-		(diameter 0)
-		(color 0 0 0 0)
-	)
-	(junction
-		(at 76.2 63.5)
 		(diameter 0)
 		(color 0 0 0 0)
@@
 	(wire
 		(pts
-			(xy 88.9 60.96) (xy 88.9 63.5)
+			(xy 88.9 60.96) (xy 88.9 68.58)
 		)
 		(stroke
@@
 	(wire
 		(pts
-			(xy 50.8 63.5) (xy 63.5 63.5)
+			(xy 50.8 68.58) (xy 63.5 68.58)
 		)
 		(stroke
@@
 	(wire
 		(pts
+			(xy 76.2 60.96) (xy 76.2 68.58)
+		)
+		(stroke
+			(width 0)
+			(type default)
+		)
+	)
+	(wire
+		(pts
 			(xy 114.3 59.69) (xy 114.3 60.96)
 		)
@@
 	(wire
 		(pts
+			(xy 101.6 71.12) (xy 101.6 68.58)
+		)
+		(stroke
+			(width 0)
+			(type default)
+		)
+	)
+	(wire
+		(pts
 			(xy 247.65 110.49) (xy 254 110.49)
 		)
@@
 	(wire
 		(pts
-			(xy 76.2 60.96) (xy 76.2 63.5)
-		)
-		(stroke
-			(width 0)
-			(type default)
-		)
-	)
-	(wire
-		(pts
 			(xy 219.71 50.8) (xy 228.6 50.8)
 		)
@@
 	(wire
 		(pts
-			(xy 63.5 63.5) (xy 76.2 63.5)
+			(xy 63.5 68.58) (xy 76.2 68.58)
 		)
 		(stroke
@@
 	(wire
 		(pts
-			(xy 88.9 68.58) (xy 88.9 63.5)
-		)
-		(stroke
-			(width 0)
-			(type default)
-		)
-	)
-	(wire
-		(pts
 			(xy 184.15 82.55) (xy 176.53 82.55)
 		)
@@
 	(wire
 		(pts
-			(xy 50.8 58.42) (xy 50.8 63.5)
+			(xy 50.8 58.42) (xy 50.8 68.58)
 		)
 		(stroke
@@
 	(wire
 		(pts
-			(xy 76.2 63.5) (xy 88.9 63.5)
+			(xy 76.2 68.58) (xy 88.9 68.58)
 		)
 		(stroke
@@
 	(wire
 		(pts
-			(xy 63.5 60.96) (xy 63.5 63.5)
+			(xy 63.5 60.96) (xy 63.5 68.58)
 		)
 		(stroke
@@
 	(symbol
 		(lib_id "power:GND")
-		(at 101.6 68.58 0)
+		(at 101.6 71.12 0)
 		(unit 1)
 		(exclude_from_sim no)
@@
 		(fields_autoplaced yes)
 		(property "Reference" "#PWR03"
-			(at 101.6 74.93 0)
+			(at 101.6 77.47 0)
 			(effects
 				(font
@@
 		)
 		(property "Value" "GND"
-			(at 101.6 73.66 0)
+			(at 101.6 76.2 0)
 			(effects
 				(font
@@
 		)
 		(property "Footprint" ""
-			(at 101.6 68.58 0)
+			(at 101.6 71.12 0)
 			(effects
 				(font
@@
 		)
 		(property "Datasheet" ""
-			(at 101.6 68.58 0)
+			(at 101.6 71.12 0)
 			(effects
 				(font
@@
 		)
 		(property "Description" "Power symbol creates a global label with name \"GND\" , ground"
-			(at 101.6 68.58 0)
-			(effects
-				(font
+			(at 101.6 71.12 0)
+			(effects
+				(font

Commit message: Error Free!
yay.
Changed lines of the file:
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@@
+	)
+	(junction
+		(at 41.91 58.42)
+		(diameter 0)
+		(color 0 0 0 0)
 	)
 	(junction
@@
 		(color 0 0 0 0)
 	)
-	(junction
-		(at 101.6 68.58)
-		(diameter 0)
-		(color 0 0 0 0)
-	)
 	(no_connect
 		(at 176.53 92.71)
@@
 	(wire
 		(pts
-			(xy 88.9 68.58) (xy 101.6 68.58)
-		)
-		(stroke
-			(width 0)
-			(type default)
-		)
-	)
-	(wire
-		(pts
 			(xy 184.15 90.17) (xy 184.15 139.7)
 		)
@@
 	(wire
 		(pts
-			(xy 48.26 58.42) (xy 40.64 58.42)
+			(xy 48.26 58.42) (xy 41.91 58.42)
 		)
 		(stroke
@@
 	(wire
 		(pts
-			(xy 101.6 71.12) (xy 101.6 68.58)
-		)
-		(stroke
-			(width 0)
-			(type default)
-		)
-	)
-	(wire
-		(pts
 			(xy 247.65 110.49) (xy 254 110.49)
 		)
@@
 	(wire
 		(pts
-			(xy 101.6 68.58) (xy 114.3 68.58)
+			(xy 88.9 68.58) (xy 114.3 68.58)
 		)
 		(stroke
@@
 		(pts
 			(xy 222.25 120.65) (xy 234.95 120.65)
+		)
+		(stroke
+			(width 0)
+			(type default)
+		)
+	)
+	(wire
+		(pts
+			(xy 41.91 58.42) (xy 40.64 58.42)
 		)
 		(stroke
@@
 	)
 	(symbol
-		(lib_id "power:GND")
-		(at 101.6 71.12 0)
-		(unit 1)
-		(exclude_from_sim no)
-		(in_bom yes)
-		(on_board yes)
-		(dnp no)
-		(fields_autoplaced yes)
-		(property "Reference" "#PWR03"
-			(at 101.6 77.47 0)
-			(effects
-				(font
-					(size 1.27 1.27)
-				)
-				(hide yes)
-			)
-		)
-		(property "Value" "GND"
-			(at 101.6 76.2 0)
-			(effects
-				(font
-					(size 1.27 1.27)
-				)
-			)
-		)
-		(property "Footprint" ""
-			(at 101.6 71.12 0)
-			(effects
-				(font
-					(size 1.27 1.27)
-				)
-				(hide yes)
-			)
-		)
-		(property "Datasheet" ""
-			(at 101.6 71.12 0)
-			(effects
-				(font
-					(size 1.27 1.27)
-				)
-				(hide yes)
-			)
-		)
-		(property "Description" "Power symbol creates a global label with name \"GND\" , ground"
-			(at 101.6 71.12 0)
-			(effects
-				(font
-					(size 1.27 1.27)
-				)
-				(hide yes)
-			)
-		)
-		(pin "1"
-		)
-		(instances
-			(project ""
-				(path "/999a87cf-6a03-4be4-a445-b5341a1dddf0/2687e2c0-9b1a-479e-99ae-d56c2ca907fb"
-					(reference "#PWR03")
-					(unit 1)
-				)
-			)
-		)
-	)
-	(symbol
 		(lib_id "easyeda2kicad:TPS55289RYQR")
 		(at 158.75 91.44 0)
@@
 					(unit 1)
 				)
+			)
+		)
+	)
+	(symbol
+		(lib_id "power:PWR_FLAG")
+		(at 41.91 58.42 180)
+		(unit 1)
+		(exclude_from_sim no)
+		(in_bom yes)
+		(on_board yes)
+		(dnp no)
+		(fields_autoplaced yes)
+		(property "Reference" "#FLG01"
+			(at 41.91 60.325 0)
+			(effects
+				(font
+					(size 1.27 1.27)
+				)
+				(hide yes)
+			)
+		)
+		(property "Value" "0V reference"
+			(at 41.91 63.5 0)
+			(effects
+				(font
+					(size 1.27 1.27)
+				)
+			)
+		)
+		(property "Footprint" ""
+			(at 41.91 58.42 0)
+			(effects
+				(font
+					(size 1.27 1.27)
+				)
+				(hide yes)
+			)
+		)
+		(property "Datasheet" "~"
+			(at 41.91 58.42 0)
+			(effects
+				(font
+					(size 1.27 1.27)
+				)
+				(hide yes)
+			)
+		)
+		(property "Description" "Special symbol for telling ERC where power comes from"
+			(at 41.91 58.42 0)
+			(effects
+				(font
+					(size 1.27 1.27)
+				)
+				(hide yes)
+			)
+		)
+		(pin "1"
+		)
+		(instances
+			(project ""
+				(path "/999a87cf-6a03-4be4-a445-b5341a1dddf0/2687e2c0-9b1a-479e-99ae-d56c2ca907fb"
+					(reference "#FLG01")
+					(unit 1)
+				)
