File: Designs/KiCAD Files/WRECtangleVersions/V4.1/Wrectangle-V4/KiCAD_Elias_version/Elias_version_4.1/Elias_version_4.1.kicad_sch (KiCad schematic)
At the start: 26 parts, among them Y1 ABS25-32.768KHZ-6-T, Y2 ABS25-32.768KHZ-6-T

Commit message: made some more edits on mcu
Other:
- sheet programmer ports: added MCO, NRST, PWR_ENn, STLK_RX, STLK_TX, SWO, TCK, TMS; removed none
Changed lines of the file:
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@@
 	)
 	(sheet
-		(at 215.9 36.83)
-		(size 58.42 40.64)
+		(at 238.76 30.48)
+		(size 36.83 40.64)
 		(exclude_from_sim no)
 		(in_bom yes)
@@
 		)
 		(property "Sheetname" "programmer"
-			(at 215.9 36.1184 0)
+			(at 238.76 29.7684 0)
 			(effects
 				(font
@@
 		)
 		(property "Sheetfile" "stm32f1_programmer.kicad_sch"
-			(at 215.9 78.0546 0)
+			(at 238.76 71.7046 0)
 			(effects
 				(font
@@
 			)
 		)
+		(pin "SWO" bidirectional
+			(at 238.76 35.56 180)
+			(effects
+				(font
+					(size 1.27 1.27)
+				)
+				(justify left)
+			)
+		)
+		(pin "PWR_ENn" output
+			(at 238.76 38.1 180)
+			(effects
+				(font
+					(size 1.27 1.27)
+				)
+				(justify left)
+			)
+		)
+		(pin "STLK_TX" output
+			(at 238.76 59.69 180)
+			(effects
+				(font
+					(size 1.27 1.27)
+				)
+				(justify left)
+			)
+		)
+		(pin "STLK_RX" input
+			(at 238.76 62.23 180)
+			(effects
+				(font
+					(size 1.27 1.27)
+				)
+				(justify left)
+			)
+		)
+		(pin "NRST" bidirectional
+			(at 238.76 52.07 180)
+			(effects
+				(font
+					(size 1.27 1.27)
+				)
+				(justify left)
+			)
+		)
+		(pin "TCK" bidirectional
+			(at 238.76 40.64 180)
+			(effects
+				(font
+					(size 1.27 1.27)
+				)
+				(justify left)
+			)
+		)
+		(pin "TMS" bidirectional
+			(at 238.76 43.18 180)
+			(effects
+				(font
+					(size 1.27 1.27)
+				)
+				(justify left)
+			)
+		)
+		(pin "MCO" bidirectional
+			(at 238.76 45.72 180)
+			(effects
+				(font
+					(size 1.27 1.27)
+				)
+				(justify left)
+			)
+		)

Commit message: made a few more edits to the mcu
Parts:
- added C10: 4.3 pF, symbol Device:C
- added JP20: SolderJumper_2_Open, symbol Jumper:SolderJumper_2_Open
- added R11: 10 K, symbol Device:R_US
Connections:
- net +3.3VP: now also FB1.2, JP20.1 (A)
- net +3.3VP_A: now also FB1.1
- net GNDREF: now also C10.2, R11.1
- net +3.3VP_bat/VLCD: now reaches U1.1 (VBAT)
- net +3.3VP_bat/VLCD: now also C10.1, JP20.2 (B)
- net TCK: now reaches U1.45 (PA12)
- net TMS: now reaches U1.46 (PA13)
- net SWO: now reaches U1.55 (PB3)
- net BOOT0: now reaches U1.60 (BOOT0)
- net BOOT0: now also R11.2
- net PH0 renamed MCO
Other:
- moved on the sheet: C1, C2, C4, C5, C6, C7, C8, FB1, JP1, JP2, JP3, JP4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
