File: Designs/KiCAD Files/WRECtangleVersions/V4.1/Wrectangle-V4/KiCAD_Elias_version/Elias_version_4.1/stm32f1_programmer.kicad_sch (KiCad schematic)
At the start: 39 parts

Commit message: made some more edits on mcu
Parts:
- added D1: D, symbol Device:D
- added J1: Conn_01x04_Pin, symbol Connector:Conn_01x04_Pin
- added J2: Conn_01x06_Pin, symbol Connector:Conn_01x06_Pin
- added JP10, JP11, JP12, JP13, JP14, JP15, JP16, JP17, JP18, JP9: SolderJumper_2_Open, symbol Jumper:SolderJumper_2_Open
- added R10: 100, symbol Device:R_US
- added R5: 10 K, symbol Device:R_US
- added R6, R7, R8, R9: 22, symbol Device:R_US
Connections:
- net +3.3VP_ST_LINK: now also JP13.2 (B), R10.2
- net GNDREF: now also J2.3 (Pin_3), JP15.2 (B), R5.2
- net STM JTMS: now also JP16.2 (B)
- net T JTCK: now also JP9.1 (A), R8.2
- net T JTMS: now also JP11.1 (A), R6.2
- net T SWO: now also JP18.1 (A), R7.2
- net OSC IN: now reaches C?.2, U2.5 (OSCIN), Y?.1
- net PWR_EXT: now reaches R?.1, R?.2, U4.1 (COMMON)
- net PWR_EXT: now also U2.39 (PB3/JTDO); no longer U2.38 (PA15/JTDI)
- net OSC OUT: now reaches C?.2, U2.6 (OSCOUT), Y?.3
- net USB_RENUMn: now reaches R?.2
- net USB_RENUMn: now also U2.38 (PA15/JTDI)
- net STM RST: now reaches C?.2, R?.1, U2.7 (NRST)
- net T_JTCK: now reaches U2.15 (PA5)
- net T_JTDO: now reaches U2.16 (PA6)
- net T_JTDI: now reaches U2.17 (PA7)
- net T_NRST: now reaches U2.18 (PB0)
- net T_JRST: now reaches U2.19 (PB1)
- net STM_JTCK: now reaches U2.37 (JTCK/SWCLK)
- net USART RX renamed STLK_RX
- net USART TX renamed STLK_TX
- new net: J1.3 (Pin_3), JP11.2 (B), JP15.1 (A)
- new net: D1.2 (A), J2.1 (Pin_1), R5.1
- new net: J2.2 (Pin_2), R8.1
- new net: J2.4 (Pin_4), R6.1
- new net: J2.5 (Pin_5), R9.1
- new net: J2.6 (Pin_6), R7.1
- new net: D1.1 (K), R10.1
- new net: J1.2 (Pin_2), JP10.2 (B), JP14.1 (A)
- new net: J1.1 (Pin_1), JP13.1 (A), JP9.2 (B)
- new net: J1.4 (Pin_4), JP12.2 (B), JP16.1 (A)
- new net NRST: JP17.2 (B)
- new net STM JTCK: JP14.2 (B)
- new net SWO: JP18.2 (B)
- new net T NRST: JP17.1 (A), R9.2
- new net TCK: JP10.1 (A)
- new net TMS: JP12.1 (A)

Commit message: made a few more edits to the mcu
Parts:
- added JP19: SolderJumper_2_Open, symbol Jumper:SolderJumper_2_Open
Connections:
- net MCO: now also JP19.2 (B); no longer C?.1, R?.2
- new net: C?.1, JP19.1 (A), R?.2
Changed lines of the file:
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@@
 	)
 	(junction
-		(at 194.31 93.98)
+		(at 132.08 176.53)
 		(diameter 0)
 		(color 0 0 0 0)
 	)
 	(junction
-		(at 132.08 176.53)
+		(at 194.31 93.98)
 		(diameter 0)
 		(color 0 0 0 0)
@@
 	(wire
 		(pts
-			(xy 172.72 96.52) (xy 205.74 96.52)
+			(xy 172.72 96.52) (xy 220.98 96.52)
 		)
 		(stroke
@@
 	(wire
 		(pts
-			(xy 194.31 93.98) (xy 205.74 93.98)
-		)
-		(stroke
-			(width 0)
-			(type default)
-		)
-	)
-	(wire
-		(pts
 			(xy 80.01 99.06) (xy 85.09 99.06)
 		)
@@
 	(wire
 		(pts
+			(xy 214.63 93.98) (xy 220.98 93.98)
+		)
+		(stroke
+			(width 0)
+			(type default)
+		)
+	)
+	(wire
+		(pts
 			(xy 224.79 45.72) (xy 227.33 45.72)
 		)
@@
 	(wire
 		(pts
+			(xy 194.31 93.98) (xy 207.01 93.98)
+		)
+		(stroke
+			(width 0)
+			(type default)
+		)
+	)
+	(wire
+		(pts
 			(xy 80.01 165.1) (xy 78.74 165.1)
 		)
@@
 	(hierarchical_label "MCO"
 		(shape bidirectional)
-		(at 205.74 93.98 0)
+		(at 220.98 93.98 0)
 		(effects
 			(font
@@
 	(hierarchical_label "PWR_ENn"
 		(shape output)
-		(at 205.74 96.52 0)
+		(at 220.98 96.52 0)
 		(effects
 			(font
@@
 					(unit 1)
 				)
+			)
+		)
+	)
+	(symbol
+		(lib_id "Jumper:SolderJumper_2_Open")
+		(at 210.82 93.98 0)
+		(unit 1)
+		(exclude_from_sim no)
+		(in_bom no)
+		(on_board yes)
+		(dnp no)
+		(property "Reference" "JP19"
+			(at 214.63 92.71 0)
+			(effects
+				(font
+					(size 1.27 1.27)
+				)
+			)
+		)
+		(property "Value" "SolderJumper_2_Open"
+			(at 210.82 90.17 0)
+			(effects
+				(font
+					(size 1.27 1.27)
+				)
+				(hide yes)
+			)
+		)
+		(property "Footprint" ""
+			(at 210.82 93.98 0)
+			(effects
+				(font
+					(size 1.27 1.27)
+				)
+				(hide yes)
+			)
+		)
+		(property "Datasheet" "~"
+			(at 210.82 93.98 0)
+			(effects
+				(font
+					(size 1.27 1.27)
+				)
+				(hide yes)
+			)
+		)
+		(property "Description" "Solder Jumper, 2-pole, open"
+			(at 210.82 93.98 0)
+			(effects
+				(font
+					(size 1.27 1.27)
+				)
+				(hide yes)
+			)
+		)
+		(pin "1"
+		)
+		(pin "2"
+		)
+		(instances
+			(project ""
+				(path "/cbbf53b7-8e33-482d-a74d-b988d551a9ab/45384e34-8109-461e-9e6e-d4eb26901d6b"
+					(reference "JP19")
+					(unit 1)
+				)
